Commit message: Add omega85 props

File: net_ft_description/urdf/net_ft_sensor_macro.urdf.xacro (robot description, xacro)
@@ -36,4 +36,10 @@
       <xacro:property name="sensor_radius" value="0.07"/>
       <xacro:property name="sensor_height" value="0.0375"/>
+    </xacro:if>
+    <xacro:if value="${sensor_type == 'ati_omega'}">
+      <xacro:property name="mesh_file" value="ati_omega_ip68_ft_sensor"/>
+      <xacro:property name="sensor_mass" value="0.5"/>
+      <xacro:property name="sensor_radius" value="0.04635"/>
+      <xacro:property name="sensor_height" value="0.03870"/>
     </xacro:if>
     <joint name="${prefix}fts_joint" type="fixed">

Commit message: correct mass

File: net_ft_description/urdf/net_ft_sensor_macro.urdf.xacro (robot description, xacro)
@@ -39,5 +39,5 @@
     <xacro:if value="${sensor_type == 'ati_omega'}">
       <xacro:property name="mesh_file" value="ati_omega_ip68_ft_sensor"/>
-      <xacro:property name="sensor_mass" value="0.5"/>
+      <xacro:property name="sensor_mass" value="1.91"/>
       <xacro:property name="sensor_radius" value="0.04635"/>
       <xacro:property name="sensor_height" value="0.03870"/>

Commit message: add pliant custom type

File: net_ft_description/urdf/net_ft_sensor_macro.urdf.xacro (robot description, xacro)
@@ -43,4 +43,10 @@
       <xacro:property name="sensor_height" value="0.03870"/>
     </xacro:if>
+    <xacro:if value="${sensor_type == 'ati_omega_pliant'}">
+      <xacro:property name="mesh_file" value="ati_omega_ip68_ft_sensor_with_clamp"/>
+      <xacro:property name="sensor_mass" value="1.91"/>
+      <xacro:property name="sensor_radius" value="0.04635"/>
+      <xacro:property name="sensor_height" value="0.03870"/>
+    </xacro:if>
     <joint name="${prefix}fts_joint" type="fixed">
       <!-- The parent link must be read from the robot model it is attached to. -->

Commit message: Fix mesh names

File: net_ft_description/urdf/net_ft_sensor_macro.urdf.xacro (robot description, xacro)
@@ -38,5 +38,5 @@
     </xacro:if>
     <xacro:if value="${sensor_type == 'ati_omega'}">
-      <xacro:property name="mesh_file" value="ati_omega_ip68_ft_sensor"/>
+      <xacro:property name="mesh_file" value="ati_omega85_ip68_ft_sensor"/>
       <xacro:property name="sensor_mass" value="1.91"/>
       <xacro:property name="sensor_radius" value="0.04635"/>
@@ -44,5 +44,5 @@
     </xacro:if>
     <xacro:if value="${sensor_type == 'ati_omega_pliant'}">
-      <xacro:property name="mesh_file" value="ati_omega_ip68_ft_sensor_with_clamp"/>
+      <xacro:property name="mesh_file" value="ati_omega85_ip68_ft_sensor_with_clamp"/>
       <xacro:property name="sensor_mass" value="1.91"/>
       <xacro:property name="sensor_radius" value="0.04635"/>

Commit message: Move inertia to correct location

File: net_ft_description/urdf/net_ft_sensor_macro.urdf.xacro (robot description, xacro)
@@ -69,5 +69,5 @@
       </collision>
       <xacro:cylinder_inertial radius="${sensor_radius}" length="${sensor_height}" mass="${sensor_mass}">
-        <xacro:insert_block name="origin" />
+        <origin xyz="0 0 ${sensor_height/2}" rpy="0 0 0"/>
       </xacro:cylinder_inertial>
     </link>
